Commit message: add grasp

File: cvgl/torus_0.urdf (robot description, URDF)
Before this commit: robot cube.urdf, 1 links, 0 joints
Links:
- link baseLink: geometry collision mesh filename=torus.obj scale=.008 .008 .008; visual mesh filename=torus.obj scale=.008 .008 .008

File: cvgl/torus_1.urdf (robot description, URDF)
Before this commit: robot cube.urdf, 1 links, 0 joints
Links:
- link baseLink: geometry collision mesh filename=torus.obj scale=.01 .01 .01; visual mesh filename=torus.obj scale=.01 .01 .01

File: cvgl/torus_2.urdf (robot description, URDF)
Before this commit: robot cube.urdf, 1 links, 0 joints
Links:
- link baseLink: geometry collision mesh filename=torus.obj scale=.016 .016 .016; visual mesh filename=torus.obj scale=.016 .016 .016

File: cvgl/torus_3.urdf (robot description, URDF)
Before this commit: robot cube.urdf, 1 links, 0 joints
Links:
- link baseLink: geometry collision mesh filename=torus.obj scale=.023 .023 .023; visual mesh filename=torus.obj scale=.023 .023 .023

File: cvgl/torus_4.urdf (robot description, URDF)
Before this commit: robot cube.urdf, 1 links, 0 joints
Links:
- link baseLink: geometry collision mesh filename=torus.obj scale=.03 .03 .03; visual mesh filename=torus.obj scale=.03 .03 .03
