Commit message: new urdf

File: cvgl/grasp/airplane1/airplane1.urdf (robot description, URDF)
Before this commit: robot cube.urdf, 1 links, 0 joints
Links:
- link baseLink: mass .02 -> 2; geometry collision mesh filename=model.obj scale=.6 .6 .6; visual mesh filename=model.obj scale=.6 .6 .6

File: cvgl/grasp/guitar/guitar.urdf (robot description, URDF)
Before this commit: robot cube.urdf, 1 links, 0 joints
Links:
- link baseLink: mass .02 -> 1.0; geometry collision mesh filename=model.obj scale=.6 .6 .6; visual mesh filename=model.obj scale=.6 .6 .6

File: cvgl/grasp/lamp1/lamp.urdf (robot description, URDF)
Before this commit: robot cube.urdf, 1 links, 0 joints
Links:
- link baseLink: mass .02 -> 1.2; geometry collision mesh filename=model.obj scale=.8 .8 .8; visual mesh filename=model.obj scale=.8 .8 .8

File: cvgl/grasp/lamp1/lamp1.urdf (robot description, URDF)
Before this commit: robot cube.urdf, 1 links, 0 joints
Links:
- link baseLink: mass .02 -> 2; geometry collision mesh filename=model.obj scale=.8 .8 .8; visual mesh filename=model.obj scale=.8 .8 .8

File: cvgl/torus_1.urdf (robot description, URDF)
Before this commit: robot cube.urdf, 1 links, 0 joints
Links:
- link baseLink: mass .02 -> .03; geometry collision mesh filename=torus.obj scale=.018 .018 .018; visual mesh filename=torus.obj scale=.018 .018 .018

File: cvgl/torus_2.urdf (robot description, URDF)
Before this commit: robot cube.urdf, 1 links, 0 joints
Links:
- link baseLink: geometry collision mesh filename=torus.obj scale=.021 .021 .021; visual mesh filename=torus.obj scale=.021 .021 .021

File: cvgl/torus_3.urdf (robot description, URDF)
Before this commit: robot cube.urdf, 1 links, 0 joints
Links:
- link baseLink: geometry collision mesh filename=torus.obj scale=.025 .025 .025; visual mesh filename=torus.obj scale=.025 .025 .025

File: cvgl/torus_4.urdf (robot description, URDF)
Before this commit: robot cube.urdf, 1 links, 0 joints
Links:
- link baseLink: geometry collision mesh filename=torus.obj scale=.015 .015 .015; collision mesh filename=torus.obj scale=.03 .03 .03
